File: KiCAD/car-control/car-control.kicad_pcb (KiCad board)
At the start: 2 copper layers, 171.4 x 40 mm, 13 parts, among them SW1 SW_Push, SW2 SW_Push, SW3 SW_Push, SW4 SW_Push, SW5 COM-15140

Commit message: working on layout
Parts:
- added A1: Arduino_MKR_Zero_Socket, PCM_arduino-library:Arduino_MKR_Zero_Socket, B.Cu at (179.1, 60.1)
- added J1: USB_B_Micro, my_USB:CONN_USB3131-30-0230-A_GCT, F.Cu at (92.6, 87.6)
- added J2: Conn_01x06, Connector_PinHeader_2.54mm:PinHeader_1x06_P2.54mm_Vertical, B.Cu at (241.9, 62.9)
- added J3: USB_A, my_USB:CONN_USB-A-S-VT_ADM, B.Cu at (94.6, 79.8)
- added J4: Conn_01x04, Connector_PinSocket_2.54mm:PinSocket_1x04_P2.54mm_Vertical, B.Cu at (187.7, 73.3)
- added R1: 10k, Resistor_SMD:R_1206_3216Metric_Pad1.30x1.75mm_HandSolder, F.Cu at (151.8, 73.7)
- added R2: 10k, Resistor_SMD:R_1206_3216Metric_Pad1.30x1.75mm_HandSolder, F.Cu at (155.6, 73.7)
- added R5: 470, Resistor_SMD:R_1206_3216Metric_Pad1.30x1.75mm_HandSolder, F.Cu at (133.3, 73.7)
- added R6: 470, Resistor_SMD:R_1206_3216Metric_Pad1.30x1.75mm_HandSolder, F.Cu at (137.8, 73.7)
- added U1: OLED-SSD1322, my_OLED:OLED_312_16pin, F.Cu at (100.3, 53.2)
- R3, R4: value 470 -> 1k; moved to F.Cu
Connections:
- net VCC renamed +3.3V
- D1 pad 1: Net-(D1-K) -> /LED0
- D2 pad 1: Net-(D2-K) -> /LED1
Routing:
- net /SW1: track 0.00 -> 117.4 mm, vias 0 -> 1
- net /A0: track 0.00 -> 104.1 mm, vias 0 -> 1
- net /A1: track 0.00 -> 101.7 mm, vias 0 -> 1
- net /SW3: track 0.00 -> 99.2 mm, vias 0 -> 1
- net /SW0: track 0.00 -> 99.2 mm, vias 0 -> 1
- net /SW2: track 0.00 -> 78.6 mm, vias 0 -> 1
- net /ENC_SW: track 0.00 -> 65.5 mm, vias 0 -> 2
- net Net-(SW5-RED): track 0.00 -> 64.1 mm, vias 0 -> 2
- net Net-(SW5-GREEN): track 0.00 -> 62.7 mm, vias 0 -> 2
- net /~{RST}: track 0.00 -> 42.2 mm, vias 0 -> 1
- net /DC: track 0.00 -> 41.0 mm, vias 0 -> 1
- net /SCK: track 0.00 -> 40.7 mm, vias 0 -> 1
- net /MOSI: track 0.00 -> 33.9 mm, vias 0 -> 1
- net /~{CS}: track 0.00 -> 27.5 mm, vias 0 -> 1
- net Net-(J1-D+): track 0.00 -> 11.8 mm
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- added copper zone on F.Cu, net +3.3V
- added copper zone on B.Cu, net GND
Other:
- board text added: "A0"
- board text added: "A1"
- board text added: "A3"
- board text added: "Arduino MKR Zero"
- board text added: "CarPuter control panel"
- board text added: "E. Hazen Rev 1.0 - 2025-09"
- board text added: "OLED DISPLAY"
- board text removed: "1"
- board text removed: "Contrast"
- board text removed: "Control Panel PCB 1.0"
- board text removed: "E. Hazen Rev 1.0 - 2024-05"
- board text removed: "RX"
- board text removed: "TX"
- board text removed: "VCC"

Commit message: working on layout, move USB
Parts:
- moved J1 151.0 mm to (243.2, 76.8), turned to -90 degrees
- moved J3 146.6 mm to (240.0, 61.6), turned to -90 degrees
- moved J2 73.4 mm to (168.9, 55.9), turned to -90 degrees
- moved R1 6.41 mm to (146.2, 76.9)
- moved R2 6.41 mm to (150.1, 76.9)
- moved R5 6.41 mm to (127.8, 76.9)
- moved R6 6.41 mm to (132.3, 76.9)
- moved A1 6.41 mm to (173.6, 63.4)
- moved U1 2.54 mm to (97.8, 53.2)
- moved J4 2.54 mm to (185.2, 73.3)
- moved D1 1.98 mm to (84.1, 52.7)
- moved D2 1.98 mm to (91.1, 52.7)
- moved R3 1.98 mm to (85.4, 57.8)
- moved R4 1.98 mm to (92.4, 57.8)
- moved SW3 1.42 mm to (212.1, 73.7)
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Routing:
- net /SW1: track 117.4 -> 0.00 mm, vias 1 -> 0
- net /A0: track 104.1 -> 0.00 mm, vias 1 -> 0
- net /A1: track 101.7 -> 0.00 mm, vias 1 -> 0
- net /SW3: track 99.2 -> 0.00 mm, vias 1 -> 0
- net /SW0: track 99.2 -> 0.00 mm, vias 1 -> 0
- net /SW2: track 78.6 -> 0.00 mm, vias 1 -> 0
- net /ENC_SW: track 65.5 -> 0.00 mm, vias 2 -> 0
- net Net-(SW5-RED): track 64.1 -> 0.00 mm, vias 2 -> 0
- net Net-(SW5-GREEN): track 62.7 -> 0.00 mm, vias 2 -> 0
- net /~{RST}: track 42.2 -> 0.00 mm, vias 1 -> 0
- net /DC: track 41.0 -> 0.00 mm, vias 1 -> 0
- net /SCK: track 40.7 -> 0.00 mm, vias 1 -> 0
- net /MOSI: track 33.9 -> 0.00 mm, vias 1 -> 0
- net /~{CS}: track 27.5 -> 0.00 mm, vias 1 -> 0
- net Net-(J1-D+): track 11.8 -> 0.00 mm
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
Commit message: PCB done?
Parts:
- added JP1: Jumper_3_Bridged12, Connector_PinHeader_2.54mm:PinHeader_1x03_P2.54mm_Vertical, B.Cu at (182.2, 61.6)
- moved J3 17.1 mm to (225.4, 70.5), turned to 0 degrees
- moved J4 9.63 mm to (180.5, 81.7), turned to -90 degrees
- moved J1 8.89 mm to (243.2, 67.9)
- moved R1 8.06 mm to (154.3, 76.9)
Connections:
- net Net-(J1-VBUS) renamed /VBUS
- A1 pad 5V: unconnected-(A1-Pad5V) -> +5V
- J4 pad 1: +3.3V -> Net-(J4-Pin_1)
Routing:
- net /SW1: track 0.00 -> 125.4 mm, vias 0 -> 1
- net /SW0: track 0.00 -> 110.1 mm, vias 0 -> 1
- net /SW3: track 0.00 -> 101.2 mm, vias 0 -> 2
- net /LED0: track 0.00 -> 89.3 mm, vias 0 -> 1
- net /SW2: track 0.00 -> 75.3 mm
- net /LED1: track 0.00 -> 73.5 mm, vias 0 -> 1
- net /ENC_SW: track 0.00 -> 66.9 mm, vias 0 -> 2
- net /RX: track 0.00 -> 65.2 mm, vias 0 -> 1
- net /TX: track 0.00 -> 64.1 mm, vias 0 -> 1
- net /VBUS: track 0.00 -> 62.7 mm
- net /ENC_A: track 0.00 -> 62.3 mm, vias 0 -> 1
- net Net-(SW5-RED): track 0.00 -> 62.0 mm, vias 0 -> 2
- net Net-(SW5-GREEN): track 0.00 -> 57.1 mm, vias 0 -> 2
- net /ENC_B: track 0.00 -> 55.5 mm, vias 0 -> 1
- net /A1: track 0.00 -> 54.1 mm, vias 0 -> 1
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Other:
- board text added: "3.3"
- board text added: "ANALOG"
- board text added: "ARDU"
- board text added: "G"
- board text added: "G Tx Rx PWR"
- board text added: "GPS PWR"
- board text added: "GPS UART"
- board text added: "VBUS"
- board text removed: "A3"
- board text removed: "GND"

Commit message: latest mount
Parts:
- moved J1 34.9 mm to (217.8, 91.7), turned to 0 degrees
- moved J3 20.2 mm to (215.9, 88.3)
- moved H4 7.75 mm to (236.9, 90.8)
- moved H3 6.35 mm to (236.9, 52.7)
- moved H2 4.45 mm to (78.1, 90.8)
Routing:
- net Net-(J1-D+): track 18.5 -> 3.99 mm
- net /VBUS: track 62.7 -> 50.1 mm
- net Net-(J1-D-): track 15.8 -> 6.71 mm
- net /SW3: track 101.2 -> 101.5 mm, vias 2 -> 0
Other:
- board size 171.4 x 40 mm -> 165.1 x 44.5 mm
