File: KiCAD/car-control/car-control.kicad_pcb (KiCad board)
At the start: 2 copper layers, 165.1 x 44.5 mm, 24 parts, among them J1 USB_B_Micro, J2 Conn_01x06, J3 USB_A, J4 Conn_01x04, SW1 SW_Push, SW2 SW_Push, SW3 SW_Push, SW4 SW_Push, SW5 COM-15140, U1 OLED-SSD1322

Commit message: initial software, fix layout
Connections:
- A1 pad D10: /MISO -> unconnected-(A1-D10_MISO-PadD10)
- U1 pad 10: unconnected-(U1-D7-Pad10) -> GND
- U1 pad 11: unconnected-(U1-FR-Pad11) -> GND
- U1 pad 12: unconnected-(U1-VDDIO-Pad12) -> GND
- U1 pad 13: unconnected-(U1-VDD-Pad13) -> GND
- U1 pad 14: GND -> /DC
- U1 pad 3: (no net) -> unconnected-(U1-NC-Pad3)
- U1 pad 4: /DC -> /SCK
- U1 pad 5: unconnected-(U1-D2-Pad5) -> /MOSI
- U1 pad 7: /MOSI -> GND
- U1 pad 8: /SCK -> GND
- U1 pad 9: unconnected-(U1-D6-Pad9) -> GND
Routing:
- net /MOSI: track 30.4 -> 24.3 mm, vias 1 -> 0
- net /DC: track 39.1 -> 33.8 mm, vias 1 -> 2
- net /SCK: track 34.5 -> 29.6 mm, vias 1 -> 0

Commit message: PCB V1.0 as built
Parts:
- J4: footprint Connector_PinSocket_2.54mm:PinSocket_1x04_P2.54mm_Vertical -> Connector_PinSocket_2.54mm:PinSocket_1x05_P2.54mm_Vertical
Connections:
- J4 pad 2: /RX -> GND
- J4 pad 3: /TX -> /RX
- J4 pad 4: GND -> /TX
Routing:
- net /RX: track 65.2 -> 64.2 mm
- net /TX: track 64.1 -> 63.4 mm
Changed lines of the file:
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@@
 	(net 38 "Net-(J4-Pin_1)")
 	(net 39 "+5V")
+	(net 40 "unconnected-(J4-Pin_5-Pad5)")
 	(footprint "my_mtg_hole:mtg_hole_4-40"
 		(layer "F.Cu")
@@
 				(keep_text_aligned yes)
 			)
-			(gr_text "3.955"
+			(gr_text "100.457"
 				(at 148.004 49.7485 0)
 				(layer "User.2")
@@
 		)
 	)
-	(footprint "Connector_PinSocket_2.54mm:PinSocket_1x04_P2.54mm_Vertical"
+	(footprint "Connector_PinSocket_2.54mm:PinSocket_1x05_P2.54mm_Vertical"
 		(layer "B.Cu")
 		(at 180.477 81.686 -90)
-		(descr "Through hole straight socket strip, 1x04, 2.54mm pitch, single row (from Kicad 4.0.7), script generated")
-		(tags "Through hole socket strip THT 1x04 2.54mm single row")
+		(descr "Through hole straight socket strip, 1x05, 2.54mm pitch, single row (from Kicad 4.0.7), script generated")
+		(tags "Through hole socket strip THT 1x05 2.54mm single row")
 		(property "Reference" "J4"
 			(at 0 2.77 90)
@@
 		)
 		(property "Value" "Conn_01x04"
-			(at 0 -10.39 90)
+			(at 0 -12.93 90)
 			(layer "B.Fab")
 			(effects
@@
 			)
 		)
-		(property "Description" "Generic connector, single row, 01x04, script generated (kicad-library-utils/schlib/autogen/connector/)"
+		(property "Description" "Generic connector, single row, 01x05, script generated (kicad-library-utils/schlib/autogen/connector/)"
 			(at 0 0 90)
 			(layer "B.Fab")
@@
 		(fp_line
 			(start -1.33 -1.27)
-			(end -1.33 -8.95)
+			(end -1.33 -11.49)
 			(stroke
 				(width 0.12)
@@
 		(fp_line
 			(start 1.33 -1.27)
-			(end 1.33 -8.95)
+			(end 1.33 -11.49)
 			(stroke
 				(width 0.12)
@@
 		)
 		(fp_line
-			(start -1.33 -8.95)
-			(end 1.33 -8.95)
+			(start -1.33 -11.49)
+			(end 1.33 -11.49)
 			(stroke
 				(width 0.12)
@@
 		(fp_line
 			(start 1.75 1.8)
-			(end 1.75 -9.4)
+			(end 1.75 -11.9)
 			(stroke
 				(width 0.05)
@@
 		)
 		(fp_line
-			(start -1.8 -9.4)
+			(start -1.8 -11.9)
 			(end -1.8 1.8)
 			(stroke
@@
 		)
 		(fp_line
-			(start 1.75 -9.4)
-			(end -1.8 -9.4)
+			(start 1.75 -11.9)
+			(end -1.8 -11.9)
 			(stroke
 				(width 0.05)
@@
 		(fp_line
 			(start 1.27 0.635)
-			(end 1.27 -8.89)
+			(end 1.27 -11.43)
 			(stroke
 				(width 0.1)
@@
 		)
 		(fp_line
-			(start -1.27 -8.89)
+			(start -1.27 -11.43)
 			(end -1.27 1.27)
 			(stroke
@@
 		)
 		(fp_line
-			(start 1.27 -8.89)
-			(end -1.27 -8.89)
+			(start 1.27 -11.43)
+			(end -1.27 -11.43)
 			(stroke
 				(width 0.1)
@@
 		)
 		(fp_text user "${REFERENCE}"
-			(at 0 -3.81 0)
+			(at 0 -5.08 180)
 			(layer "B.Fab")
 			(effects
@@
 			(layers "*.Cu" "*.Mask")
 			(remove_unused_layers no)
-			(net 21 "/RX")
+			(net 2 "GND")
 			(pinfunction "Pin_2")
 			(pintype "passive")
@@
 			(layers "*.Cu" "*.Mask")
 			(remove_unused_layers no)
-			(net 16 "/TX")
+			(net 21 "/RX")
 			(pinfunction "Pin_3")
 			(pintype "passive")
@@
 			(layers "*.Cu" "*.Mask")
 			(remove_unused_layers no)
-			(net 2 "GND")
+			(net 16 "/TX")
 			(pinfunction "Pin_4")
 			(pintype "passive")
 		)
+		(pad "5" thru_hole circle
+			(at 0 -10.16 270)
+			(size 1.7 1.7)
+			(drill 1)
+			(layers "*.Cu" "*.Mask")
+			(remove_unused_layers no)
+			(net 40 "unconnected-(J4-Pin_5-Pad5)")
+			(pinfunction "Pin_5")
+			(pintype "passive+no_connect")
+		)
 		(embedded_fonts no)
-		(model "${KICAD9_3DMODEL_DIR}/Connector_PinSocket_2.54mm.3dshapes/PinSocket_1x04_P2.54mm_Vertical.step"
+		(model "${KICAD9_3DMODEL_DIR}/Connector_PinSocket_2.54mm.3dshapes/PinSocket_1x05_P2.54mm_Vertical.step"
 			(offset
 				(xyz 0 0 0)
@@
 			(keep_text_aligned yes)
 		)
-		(gr_text "6.2500 in"
+		(gr_text "158.7500 mm"
 			(at 157.48 104.387 0)
 			(layer "User.2")
@@
 			(keep_text_aligned yes)
 		)
-		(gr_text "1.7500 in"
+		(gr_text "44.4500 mm"
 			(at 60.064 71.755 90)
 			(layer "User.2")
@@
 			(keep_text_aligned yes)
 		)
-		(gr_text "0.1250 in"
+		(gr_text "3.1750 mm"
 			(at 65.906 51.1175 90)
 			(layer "User.2")
@@
 			(keep_text_aligned yes)
 		)
-		(gr_text "0.1250 in"
+		(gr_text "3.1750 mm"
 			(at 238.4425 37.712 0)
 			(layer "User.2")
@@
 			(keep_text_aligned yes)
 		)
-		(gr_text "0.1250 in"
+		(gr_text "3.1750 mm"
 			(at 76.5175 37.458 0)
 			(layer "User.2")
@@
 			(keep_text_aligned yes)
 		)
-		(gr_text "6.5000 in"
+		(gr_text "165.1000 mm"
 			(at 157.48 25.393 0)
 			(layer "User.2")
@@
 			(keep_text_aligned yes)
 		)
-		(gr_text "1.5000 in"
+		(gr_text "38.1000 mm"
 			(at 62.096 71.755 90)
 			(layer "User.2")
@@
 	)
 	(segment
+		(start 188.097 79.893)
+		(end 188.097 81.686)
+		(width 0.254)
+		(layer "F.Cu")
+		(net 16)
+	)
+	(segment
 		(start 187.706 66.421)
+		(end 187.706 79.502)
+		(width 0.254)
+		(layer "F.Cu")
+		(net 16)
+	)
+	(segment
+		(start 187.706 79.502)
 		(end 187.706 79.537)
 		(width 0.254)
@@
 	)
 	(segment
-		(start 187.706 79.537)
-		(end 185.557 81.686)
+		(start 187.706 79.502)
+		(end 188.097 79.893)
 		(width 0.254)
 		(layer "F.Cu")
@@
 	)
 	(segment
-		(start 186.436 78.267)
-		(end 183.017 81.686)
+		(start 186.436 80.807)
+		(end 185.557 81.686)
 		(width 0.254)
 		(layer "F.Cu")
@@
 	(segment
 		(start 186.436 67.564)
-		(end 186.436 78.267)
+		(end 186.436 80.807)
 		(width 0.254)
 		(layer "F.Cu")
